File: MeasureVccUsingVrefBubbleDisplay/MeasureVccUsingVrefBubbleDisplay/BubbleDisplayTempSensingThermistorWithRCfilterOpampSignalConditioning.sch (EAGLE design)
At the start: 24 parts, among them IC1 ATMEGA328-20P, U1 SN74HC595N, Y1 16MHz

Commit message: Added a JobList to outline jobs completed, to be completed and known bugs. Added schematic to show connections for LM35 temperature sensor used for calibration of the thermistor sensing circuitry. Removed extra folder of Thermistor4c for Bubble Display
Parts:
- added C12, C13, C14: 0.1uF, SparkFun-Capacitors:CAPEZ
- added MCP1: (no value), Microchip_MCP6001R:MCP6001R
- added R8: 100K, SparkFun-Passives:RESISTORPTH-1/2W
- C10, C8, C9: value (none) -> 0.1uF
- C6: value (none) -> 1uF
Connections:
- new net N$13: C6.1, MCP1.VIN+, R8.1
- new net N$14: IC1.(PCI8/ADC0)PC0, MCP1.VIN-, MCP1.VOUT
- net GND: now also C10.2, C11.2, C12.2, C13.2, C14.2, C6.2, C7.2, C8.1, C9.1, MCP1.VSS; no longer C11.1
- net N$4: now also C8.2; no longer C11.2
- net N$8: now also R8.2; no longer IC1.(PCI8/ADC0)PC0
- net VCC: now also C10.1, C11.1, C12.1, C13.1, C14.1, C7.1, C9.2, MCP1.VDD
Other:
- note added: "Thermistor Low Pass Filter Time Constant 0.1s Op-Amp Rail to Rail Input/Output Buffer"
- moved on the sheet: C10, C11, C6, C7, C8, C9, R1, R2
